File: CANNONBALL.kicad_sch (KiCad schematic)
At the start: 61 parts, among them J3 JST-PH 2.0 BATTERY, J4 I2C_CONN, J5 LEFT_PINS, J6 RIGHT_PINS, Q1 FS8205A, Q2 DMG2301L, SW1 SW_Push, U1 USBLC6-4SC6, U10 MAX17048, U2 AP2112K-3.3, U3 ESP32-C3-WROOM-02, U4 LSM6DS3, U5 DW01A, U6 BQ24075RGT, U7 SHT40, U8 VEML6030

Commit message: Add production_files to gitignore and update design files
Co-Authored-By: Claude Sonnet 4.6 <noreply@anthropic.com>
Parts:
- removed C2, C7: 100nF, Capacitor_SMD:C_0603_1608Metric_Pad1.08x0.95mm_HandSolder, symbol Device:C_Small
- removed D1: 1N5819W, diode:SOD-123_L2.7-W1.6-LS3.7-RD, symbol diode:1N5819W_C963381
- removed F1: MF-FSMF050X-2, power:F0603, symbol power:MF-FSMF050X-2
- removed Q2: DMG2301L, Package_TO_SOT_SMD:SOT-23, symbol Transistor_FET:DMG2301L
- removed R9: 10K, Resistor_SMD:R_0402_1005Metric_Pad0.72x0.64mm_HandSolder, symbol Device:R_Small
- added D2: MS2A40LWS, diode:SOD-323_L1.7-W1.25-LS2.5-RD, symbol diode:MS2A40LWS_C7380001
- added F2: 0805L110/16WR, power:F0805, symbol power:0805L110-16WR_C47345575
- added Q3: 2N7002K, Package_TO_SOT_SMD:SOT-23, symbol Transistor_FET:2N7002K
- C1: value 10uF -> 1uF
- C10, C11, C14, C16, C18, C19, C20, C21, C22, C23, C24, C3: value 100nF -> 1uF
- C15, C6: value 10uF -> 4.7uF
- R8: value 330 -> 10K
- U6: value BQ24075RGT -> TI BQ24075RGTR
Connections:
- net LED_3V3 is gone; now on net 5V: C19.2, C23.2, LED1.1 (VDD), LED2.1 (VDD)
- net 3V3: now also J4.2; no longer J4.3
- net 5V: now also D2.1 (C)
- net GND: now also J4.1, R8.1, USB1.13 (EH), USB1.14 (EH), Q3.2 (S); no longer J4.4, LED1.3 (GND), LED2.3 (GND)
- net GPIO 0 / SCL: now also J4.4; no longer J4.1
- net GPIO 1 / SDA: now also J4.3; no longer J4.2
- net GPIO 4: now also LED1.4 (DIN); no longer R8.2
- net GPIO 5: now also R8.2, Q3.1 (G)
- net VBUS: now also F2.1
- net at C1.2: now also D2.2 (A), F2.2
- new net LED_GND: LED1.3 (GND), LED2.3 (GND), Q3.3 (D)
- no-connect marks 12 -> 10
Other:
- moved on the sheet: R14, R15, R2, R3, R6, R7, SW1, U3, U4, U8
